Commit message: sync730

File: src/mjlab/asset_zoo/robots/RL_BOY/RLBOY.urdf (robot description, URDF)
Before this commit: robot RL_BOY, 21 links, 20 joints
Joints:
- joint left_knee_pitch_joint: limit lower=0 upper=2.2 effort=21 velocity=21 -> lower=-0.1 upper=2.2 effort=21 velocity=21
- joint left_shoulder_roll_joint: limit lower=-0.2 upper=1.5 effort=5 velocity=21 -> lower=-0.2 upper=2.0 effort=5 velocity=21
- joint right_knee_pitch_joint: limit lower=0 upper=2.2 effort=21 velocity=21 -> lower=-0.1 upper=2.2 effort=21 velocity=21
- joint right_shoulder_roll_joint: limit lower=-1.5 upper=0.2 effort=5 velocity=21 -> lower=-2.0 upper=0.2 effort=5 velocity=21
