Commit message: addQL2.0

File: src/mjlab/asset_zoo/robots/QLmini2.0/urdf/qinglongmini2.0.urdf (robot description, URDF)
Before this commit: robot qinglongmini2.0, 20 links, 19 joints
Links:
- link base_link: geometry collision cylinder length=0.1 radius=0.05; visual mesh filename=../meshes/base_link.STL
- link left_elbow_link: geometry collision cylinder length=0.12 radius=0.02; collision sphere radius=0.02
- link left_foot: geometry collision box size=0.08 0.06 0.02; collision cylinder length=0.02 radius=0.03
- link left_hip_pitch_link: geometry collision box size=0.08 0.07 0.12; visual mesh filename=../meshes/left_hip_pitch_link.STL
- link left_hip_roll_link: geometry collision cylinder length=0.06 radius=0.035; visual mesh filename=../meshes/left_hip_roll_link.STL
- link left_hip_yaw_link: geometry collision cylinder length=0.07 radius=0.04; visual mesh filename=../meshes/left_hip_yaw_link.STL
- link left_knee_link: geometry collision box size=0.09 0.08 0.20; visual mesh filename=../meshes/left_knee_link.STL
- link left_shoulder_pitch_link: geometry collision cylinder length=0.07 radius=0.03; visual mesh filename=../meshes/left_shoulder_pitch_link.STL
- link left_shoulder_roll_link: geometry collision cylinder length=0.06 radius=0.03; visual mesh filename=../meshes/left_shoulder_roll_link.STL
- link left_shoulder_yaw_link: geometry collision cylinder length=0.07 radius=0.028; visual mesh filename=../meshes/left_shoulder_yaw_link.STL
- link right_elbow_link: geometry collision cylinder length=0.12 radius=0.02; collision sphere radius=0.02
- link right_foot: geometry collision box size=0.08 0.06 0.02; collision cylinder length=0.02 radius=0.03
- link right_hip_pitch_link: geometry collision box size=0.08 0.07 0.12; visual mesh filename=../meshes/right_hip_pitch_link.STL
- link right_hip_roll_link: geometry collision cylinder length=0.06 radius=0.035; visual mesh filename=../meshes/right_hip_roll_link.STL
- link right_hip_yaw_link: geometry collision cylinder length=0.07 radius=0.04; visual mesh filename=../meshes/right_hip_yaw_link.STL
- link right_knee_link: geometry collision box size=0.09 0.08 0.20; visual mesh filename=../meshes/right_knee_link.STL
- link right_shoulder_pitch_link: geometry collision cylinder length=0.07 radius=0.03; visual mesh filename=../meshes/right_shoulder_pitch_link.STL
- link right_shoulder_roll_link: geometry collision cylinder length=0.06 radius=0.03; visual mesh filename=../meshes/right_shoulder_roll_link.STL
- link right_shoulder_yaw_link: geometry collision cylinder length=0.07 radius=0.028; visual mesh filename=../meshes/right_shoulder_yaw_link.STL
- link waist_yaw_link: geometry collision box size=0.11 0.18 0.20; visual mesh filename=../meshes/waist_yaw_link.STL
