Commit message: Update qlmini2 mass and inertia parameters

File: src/mjlab/asset_zoo/robots/qlmini2/urdf/qlmini2.urdf (robot description, URDF)
Before this commit: robot qlmini2, 20 links, 19 joints
Links:
- link base_link: mass 1.6520541 -> 1.6864
- link left_elbow_link: mass 0.1977884 -> 0.1747
- link left_foot: mass 0.251342032302528 -> 0.4411
- link left_hip_pitch_link: mass 0.5798661 -> 0.6373
- link left_hip_roll_link: mass 0.5591978 -> 0.5982
- link left_hip_yaw_link: mass 0.5211244 -> 0.5783
- link left_knee_link: mass 0.8775823 -> 0.9700
- link left_shoulder_pitch_link: mass 0.2947554 -> 0.3076
- link left_shoulder_roll_link: mass 0.3485680 -> 0.370
- link left_shoulder_yaw_link: mass 0.2995524 -> 0.3175
- link right_elbow_link: mass 0.1977884 -> 0.1747
- link right_foot: mass 0.251342026054478 -> 0.4411
- link right_hip_pitch_link: mass 0.5798660 -> 0.6373
- link right_hip_roll_link: mass 0.5591978 -> 0.5982
- link right_hip_yaw_link: mass 0.5211244 -> 0.5783
- link right_knee_link: mass 0.8775823 -> 0.9700
- link right_shoulder_pitch_link: mass 0.2947553 -> 0.3076
- link right_shoulder_roll_link: mass 0.3485680 -> 0.370
- link right_shoulder_yaw_link: mass 0.2995524 -> 0.3175
- link waist_yaw_link: mass 3.6534181 -> 3.7654
